File: hardware/power.kicad_sch (KiCad schematic)
At the start: 6 parts, among them SW1 JS102011SAQN, U1 BQ25895RTWR, U2 TPS62840DLYR, U3 TPS61088RHLR, U4 TPS63020DSJR, U5 BQ25504RGTR

Commit message: schematic: capture 10 sensor/power/io BOM line items into the schematic layer (20/62 -> 30/62)
Adds U19-U28 with datasheet-anchored footprints and REAL sourced LCSC part
numbers (verified 2026-11-02): TPS22918DBVR, INA3221AIRGVR, BQ27441-G1A,
TPS2051BDBVR (power); BMA400, BMP390, TMP112AIDRLR (compute); TUSB320RWBR,
TXU0104PWR, MAX98357A (io).

Files moved in lockstep: .kicad_sch symbol blocks, netlist comps, BOM CSV rows,
CPL centroids (inside 222x160 board), kicad_pcb fp_text reference labels
(reference-grade single pads per U5/U14 convention; full pad maps and routing
remain the stated 'unrouted PCB' phase).

scripts/capture_schematic_parts.py is the generator + assert (Phase 11 contract:
netlist == BOM == CPL == 30 designators). spec_values schematic_coverage_baseline
20 -> 30; prose in README/BOM/HANDOFF normalized; STATUS.md regenerated.

Co-Authored-By: DeepSeek V4-Flash 0731 <noreply@anthropic.com>
Harness: pi (openrouter/deepseek/deepseek-v4-flash-0731, session 01a15a7c)
Parts:
- added U19: TPS22918DBVR, Package_TO_SOT_SMD:SOT-23-6, symbol SolarDeck_Power:TPS22918DBVR
- added U20: INA3221AIRGVR, Package_DFN_QFN:VQFN-16-1EP_4x4mm_P0.65mm, symbol SolarDeck_Power:INA3221AIRGVR
- added U21: BQ27441-G1A, Package_DFN_QFN:VSON-12_2.5x4mm_P0.5mm, symbol SolarDeck_Power:BQ27441-G1A
- added U22: TPS2051BDBVR, Package_TO_SOT_SMD:SOT-23-5, symbol SolarDeck_Power:TPS2051BDBVR
Changed lines of the file:
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@@
   (hierarchical_label "CHEM_SEL_RP" (shape output) (at 50.8 114.3 0))
   (hierarchical_label "SOLAR_ADC_IN" (shape output) (at 241.3 121.92 0))
+  ;; U19: TPS22918DBVR (Ultra-Low Leakage Load Switch)
+  (symbol (lib_id "SolarDeck_Power:TPS22918DBVR") (at 150.0 135.0 0) (unit 1)
+    (in_bom yes) (on_board yes) (dnp no)
+    (property "Reference" "U19" (at 150.0 125.0 0) (effects (font (size 1.27 1.27))))
+    (property "Value" "TPS22918DBVR" (at 150.0 127.5 0) (effects (font (size 1.27 1.27))))
+    (property "Footprint" "Package_TO_SOT_SMD:SOT-23-6" (at 150.0 135.0 0) (effects (font (size 1.27 1.27)) hide))
+    (property "Datasheet" "https://www.ti.com/lit/ds/symlink/tps22918.pdf" (at 150.0 135.0 0) (effects (font (size 1.27 1.27)) hide))
+    (property "Description" "Ultra-Low Leakage Load Switch (LTE/Wi-Fi/Audio/Exp rail gate, I_off<25mW S2idle)" (at 150.0 135.0 0) (effects (font (size 1.27 1.27)) hide))
+  )
+  ;; U20: INA3221AIRGVR (3-Channel High-Side Current & Power Monitor)
+  (symbol (lib_id "SolarDeck_Power:INA3221AIRGVR") (at 170.0 135.0 0) (unit 1)
+    (in_bom yes) (on_board yes) (dnp no)
+    (property "Reference" "U20" (at 170.0 125.0 0) (effects (font (size 1.27 1.27))))
+    (property "Value" "INA3221AIRGVR" (at 170.0 127.5 0) (effects (font (size 1.27 1.27))))
+    (property "Footprint" "Package_DFN_QFN:VQFN-16-1EP_4x4mm_P0.65mm" (at 170.0 135.0 0) (effects (font (size 1.27 1.27)) hide))
+    (property "Datasheet" "https://www.ti.com/lit/ds/symlink/ina3221.pdf" (at 170.0 135.0 0) (effects (font (size 1.27 1.27)) hide))
+    (property "Description" "3-Channel High-Side Current & Power Monitor (rail telemetry)" (at 170.0 135.0 0) (effects (font (size 1.27 1.27)) hide))
+  )
+  ;; U21: BQ27441-G1A (Impedance Track Battery Fuel Gauge & Health)
+  (symbol (lib_id "SolarDeck_Power:BQ27441-G1A") (at 150.0 150.0 0) (unit 1)
+    (in_bom yes) (on_board yes) (dnp no)
+    (property "Reference" "U21" (at 150.0 140.0 0) (effects (font (size 1.27 1.27))))
+    (property "Value" "BQ27441-G1A" (at 150.0 142.5 0) (effects (font (size 1.27 1.27))))
+    (property "Footprint" "Package_DFN_QFN:VSON-12_2.5x4mm_P0.5mm" (at 150.0 150.0 0) (effects (font (size 1.27 1.27)) hide))
+    (property "Datasheet" "https://www.ti.com/lit/ds/symlink/bq27441-g1a.pdf" (at 150.0 150.0 0) (effects (font (size 1.27 1.27)) hide))
+    (property "Description" "Impedance Track Battery Fuel Gauge & Health (SOH/ESR)" (at 150.0 150.0 0) (effects (font (size 1.27 1.27)) hide))
+  )
+  ;; U22: TPS2051BDBVR (1.5A Current-Limited USB Host Distribution Power Switch)
+  (symbol (lib_id "SolarDeck_Power:TPS2051BDBVR") (at 170.0 150.0 0) (unit 1)
+    (in_bom yes) (on_board yes) (dnp no)
+    (property "Reference" "U22" (at 170.0 140.0 0) (effects (font (size 1.27 1.27))))
+    (property "Value" "TPS2051BDBVR" (at 170.0 142.5 0) (effects (font (size 1.27 1.27))))
+    (property "Footprint" "Package_TO_SOT_SMD:SOT-23-5" (at 170.0 150.0 0) (effects (font (size 1.27 1.27)) hide))
+    (property "Datasheet" "https://www.ti.com/lit/ds/symlink/tps2051.pdf" (at 170.0 150.0 0) (effects (font (size 1.27 1.27)) hide))
+    (property "Description" "1.5A Current-Limited USB Host Distribution Power Switch" (at 170.0 150.0 0) (effects (font (size 1.27 1.27)) hide))
+  )
 )

Commit message: schematic: capture 10 more BOM line items (30/62 -> 40/62) with real LCSC numbers
Batch 2: STUSB4500QTR (PD sink), BQ29700DSET (battery PCM), LM66100DCKR (VBUS
OR-ing), PN5321A3HN (NFC + crypto signer), TPD4E05U06 (ESD TVS), dual
SPH0645LM4H-B (MEMS beamforming pair at 65mm), E22-900M22S (LoRa), PCM5102APWR
(headphone DAC), DRV2605LDGST (haptic).

Footprints datasheet-anchored, incl. corrections the searches caught (TPD4E05
is USON-10 not SOT-23-6, LM66100 is SC-70-6, PCM5102A is TSSOP-20, DRV2605L is
VSSOP-10). capture_schematic_parts.py now also emits kicad_pcb footprint blocks
(reference-grade single pad per U5/U14 convention) and is fully idempotent.
Phase 11 guard extended: live prose restatements must match the netlist.

spec_values baseline 30 -> 40; README/HANDOFF prose normalized; STATUS regenerated.

Co-Authored-By: DeepSeek V4-Flash 0731 <noreply@anthropic.com>
Harness: pi (openrouter/deepseek/deepseek-v4-flash-0731, session 01a15a7c)
Parts:
- added U29: STUSB4500QTR, Package_DFN_QFN:VQFN-24-1EP_4x4mm_P0.5mm, symbol SolarDeck_Power:STUSB4500QTR
- added U31: BQ29700DSET, Package_DFN_QFN:WSON-6_1.5x1.5mm_P0.5mm, symbol SolarDeck_Power:BQ29700DSET
- added U32: LM66100DCKR, Package_TO_SOT_SMD:SC-70-6, symbol SolarDeck_Power:LM66100DCKR
Changed lines of the file:
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@@
     (property "Description" "1.5A Current-Limited USB Host Distribution Power Switch" (at 170.0 150.0 0) (effects (font (size 1.27 1.27)) hide))
   )
+  ;; U29: STUSB4500QTR (Standalone USB-PD 20W Sink Controller)
+  (symbol (lib_id "SolarDeck_Power:STUSB4500QTR") (at 190.0 135.0 0) (unit 1)
+    (in_bom yes) (on_board yes) (dnp no)
+    (property "Reference" "U29" (at 190.0 125.0 0) (effects (font (size 1.27 1.27))))
+    (property "Value" "STUSB4500QTR" (at 190.0 127.5 0) (effects (font (size 1.27 1.27))))
+    (property "Footprint" "Package_DFN_QFN:VQFN-24-1EP_4x4mm_P0.5mm" (at 190.0 135.0 0) (effects (font (size 1.27 1.27)) hide))
+    (property "Datasheet" "https://www.st.com/resource/en/datasheet/stusb4500.pdf" (at 190.0 135.0 0) (effects (font (size 1.27 1.27)) hide))
+    (property "Description" "Standalone USB-PD 20W Sink Controller (9V/12V contract, dead-battery mode)" (at 190.0 135.0 0) (effects (font (size 1.27 1.27)) hide))
+  )
+  ;; U31: BQ29700DSET (Battery Protection IC)
+  (symbol (lib_id "SolarDeck_Power:BQ29700DSET") (at 190.0 150.0 0) (unit 1)
+    (in_bom yes) (on_board yes) (dnp no)
+    (property "Reference" "U31" (at 190.0 140.0 0) (effects (font (size 1.27 1.27))))
+    (property "Value" "BQ29700DSET" (at 190.0 142.5 0) (effects (font (size 1.27 1.27))))
+    (property "Footprint" "Package_DFN_QFN:WSON-6_1.5x1.5mm_P0.5mm" (at 190.0 150.0 0) (effects (font (size 1.27 1.27)) hide))
+    (property "Datasheet" "https://www.ti.com/lit/ds/symlink/bq29700.pdf" (at 190.0 150.0 0) (effects (font (size 1.27 1.27)) hide))
+    (property "Description" "Battery Protection IC (PCM; li-ion OVP 4.275V - see ADR on LiFePO4 profile)" (at 190.0 150.0 0) (effects (font (size 1.27 1.27)) hide))
+  )
+  ;; U32: LM66100DCKR (Low-IQ Ideal-Diode VBUS OR-ing Controller)
+  (symbol (lib_id "SolarDeck_Power:LM66100DCKR") (at 190.0 145.0 0) (unit 1)
+    (in_bom yes) (on_board yes) (dnp no)
+    (property "Reference" "U32" (at 190.0 135.0 0) (effects (font (size 1.27 1.27))))
+    (property "Value" "LM66100DCKR" (at 190.0 137.5 0) (effects (font (size 1.27 1.27))))
+    (property "Footprint" "Package_TO_SOT_SMD:SC-70-6" (at 190.0 145.0 0) (effects (font (size 1.27 1.27)) hide))
+    (property "Datasheet" "https://www.ti.com/lit/ds/symlink/lm66100.pdf" (at 190.0 145.0 0) (effects (font (size 1.27 1.27)) hide))
+    (property "Description" "Low-IQ Ideal-Diode VBUS OR-ing Controller (dual, 2A)" (at 190.0 145.0 0) (effects (font (size 1.27 1.27)) hide))
+  )
 )
