File: hardware/compute.kicad_sch (KiCad schematic)
At the start: 6 parts, among them J1 DF40C-100DS-0.4V, J2 DF40C-100DS-0.4V, U10 W25Q128JVS, U11 DS3231MZ+, U8 RP2350B, U9 APS6404L-3SQR-SN

Commit message: schematic: capture 10 sensor/power/io BOM line items into the schematic layer (20/62 -> 30/62)
Adds U19-U28 with datasheet-anchored footprints and REAL sourced LCSC part
numbers (verified 2026-11-02): TPS22918DBVR, INA3221AIRGVR, BQ27441-G1A,
TPS2051BDBVR (power); BMA400, BMP390, TMP112AIDRLR (compute); TUSB320RWBR,
TXU0104PWR, MAX98357A (io).

Files moved in lockstep: .kicad_sch symbol blocks, netlist comps, BOM CSV rows,
CPL centroids (inside 222x160 board), kicad_pcb fp_text reference labels
(reference-grade single pads per U5/U14 convention; full pad maps and routing
remain the stated 'unrouted PCB' phase).

scripts/capture_schematic_parts.py is the generator + assert (Phase 11 contract:
netlist == BOM == CPL == 30 designators). spec_values schematic_coverage_baseline
20 -> 30; prose in README/BOM/HANDOFF normalized; STATUS.md regenerated.

Co-Authored-By: DeepSeek V4-Flash 0731 <noreply@anthropic.com>
Harness: pi (openrouter/deepseek/deepseek-v4-flash-0731, session 01a15a7c)
Parts:
- added U23: BMA400, Package_LGA:LGA-12_2x2mm_P0.5mm, symbol SolarDeck_Compute:BMA400
- added U24: BMP390, Package_LGA:LGA-10_2x2mm_P0.5mm, symbol SolarDeck_Compute:BMP390
- added U25: TMP112AIDRLR, Package_TO_SOT_SMD:SOT-563, symbol SolarDeck_Compute:TMP112AIDRLR
Changed lines of the file:
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@@
   (hierarchical_label "CM4_USB_DP" (shape bidirectional) (at 101.6 96.52 0))
   (hierarchical_label "CM4_USB_DM" (shape bidirectional) (at 101.6 99.06 0))
+  ;; U23: BMA400 (3-Axis Accelerometer, 3.5uA pick-up wake)
+  (symbol (lib_id "SolarDeck_Compute:BMA400") (at 20.0 60.0 0) (unit 1)
+    (in_bom yes) (on_board yes) (dnp no)
+    (property "Reference" "U23" (at 20.0 50.0 0) (effects (font (size 1.27 1.27))))
+    (property "Value" "BMA400" (at 20.0 52.5 0) (effects (font (size 1.27 1.27))))
+    (property "Footprint" "Package_LGA:LGA-12_2x2mm_P0.5mm" (at 20.0 60.0 0) (effects (font (size 1.27 1.27)) hide))
+    (property "Datasheet" "https://www.bosch-sensortec.com/media/boschsensortec/downloads/datasheets/smart-motion/bst-bma400-ds000.pdf" (at 20.0 60.0 0) (effects (font (size 1.27 1.27)) hide))
+    (property "Description" "3-Axis Accelerometer, 3.5uA pick-up wake (BMA400)" (at 20.0 60.0 0) (effects (font (size 1.27 1.27)) hide))
+  )
+  ;; U24: BMP390 (Precision Barometric Pressure & Altimeter)
+  (symbol (lib_id "SolarDeck_Compute:BMP390") (at 35.0 60.0 0) (unit 1)
+    (in_bom yes) (on_board yes) (dnp no)
+    (property "Reference" "U24" (at 35.0 50.0 0) (effects (font (size 1.27 1.27))))
+    (property "Value" "BMP390" (at 35.0 52.5 0) (effects (font (size 1.27 1.27))))
+    (property "Footprint" "Package_LGA:LGA-10_2x2mm_P0.5mm" (at 35.0 60.0 0) (effects (font (size 1.27 1.27)) hide))
+    (property "Datasheet" "https://www.bosch-sensortec.com/media/boschsensortec/downloads/datasheets/bst-bmp390-ds000.pdf" (at 35.0 60.0 0) (effects (font (size 1.27 1.27)) hide))
+    (property "Description" "Precision Barometric Pressure & Altimeter (BMP390)" (at 35.0 60.0 0) (effects (font (size 1.27 1.27)) hide))
+  )
+  ;; U25: TMP112AIDRLR (Precision Digital Temperature Sensor)
+  (symbol (lib_id "SolarDeck_Compute:TMP112AIDRLR") (at 50.0 60.0 0) (unit 1)
+    (in_bom yes) (on_board yes) (dnp no)
+    (property "Reference" "U25" (at 50.0 50.0 0) (effects (font (size 1.27 1.27))))
+    (property "Value" "TMP112AIDRLR" (at 50.0 52.5 0) (effects (font (size 1.27 1.27))))
+    (property "Footprint" "Package_TO_SOT_SMD:SOT-563" (at 50.0 60.0 0) (effects (font (size 1.27 1.27)) hide))
+    (property "Datasheet" "https://www.ti.com/lit/ds/symlink/tmp112.pdf" (at 50.0 60.0 0) (effects (font (size 1.27 1.27)) hide))
+    (property "Description" "Precision Digital Temperature Sensor (battery + display backplane)" (at 50.0 60.0 0) (effects (font (size 1.27 1.27)) hide))
+  )
 )

Commit message: AUDIT 6 + README rewrite; standardize on CM5, Kaleido 4, SGP.22 eSIM
Class: C1 CLAIM + C4 HYGIENE (spans C2 for the overlay/identifier rename).

- docs/AUDIT_6_2026-10-21.md: repo checked against datasheets. Blockers: BQ25895
  cannot charge LiFePO4 (VREG floor 3.84 V, default 4.208 V); protector and gauge are
  Li-ion parts; CM4/CM5 have no RAM-retaining low-power state; panel/stack/cell do
  not close; schematic has no connectivity; ~half the LCSC numbers are wrong.
- README.md rewritten: intent first, pillars with real status, one status section.
- ADR-031 CM5116064 is the compute standard; ADR-032 Kaleido 4 is the only panel,
  V1 waits for release (supersedes ADR-030 two-SKU); ADR-033 soldered eSIM kept,
  must be consumer SGP.22 (ST4SIM-200M rejected).
- spec_values: panel facts, reader geometry, refresh timings, epdc_spi_mhz -> null;
  CM5 supply keys; BCM2712 (was BCM2718); BOM total re-derived as a floor.
- Gates: two dead BANNED regexes fixed (red-controlled); Phase 9 accepts any
  harness attribution and no longer claims link checking; Phases 5/10 skip null
  panel facts with an UNVERIFIED line; Phase 14 counts TBD rows; Phase 16 checks
  the CM5 commitment is stated as unpublished.
- Sweep: CM4 -> CM5 across live docs, firmware identifiers, nets, production
  guides; overlay renamed solardeck-cm5.dts and marked not yet valid (RP1 port).
- Airgap switch: ties CM5 WL_nDisable/BT_nDisable low (CM5 datasheet 2.1.1-2.1.2).

verify_all.py: 16/16 green. Still unmeasured: everything.

Co-Authored-By: Claude Opus 5.5 <noreply@anthropic.com>
Harness: claude-code (anthropic/claude-opus-5-5, session f5d955c0)
Claude-Session: https://claude.ai/code/session_01CkqVCXjctA16Vs1i2pskTP
Changed lines of the file:
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@@
     (company "SolarDeck Open Hardware")
     (comment 1 "Written 2026-10-19 08:15 UTC in the Pi harness by antigravity/gemini-3.8-flash")
-    (comment 2 "Hirose DF40 CM4 + RP2350B + 8MB PSRAM + 16MB Flash + DS3231 RTC")
+    (comment 2 "Hirose DF40 CM5 + RP2350B + 8MB PSRAM + 16MB Flash + DS3231 RTC")
   )
-  ;; J1: Hirose DF40C-100DS-0.4V (CM4 Board-to-Board Socket 1)
+  ;; J1: Hirose DF40C-100DS-0.4V (CM5 Board-to-Board Socket 1)
   (symbol (lib_id "SolarDeck_Compute:Hirose_DF40C_100DS") (at 76.2 88.9 0) (unit 1)
     (in_bom yes) (on_board yes) (dnp no)
@@
     (property "Value" "DF40C-100DS-0.4V" (at 76.2 40.64 0) (effects (font (size 1.27 1.27))))
     (property "Footprint" "Connector_Hirose:Hirose_DF40C-100DS-0.4V_2x50_P0.40mm_Vertical" (at 76.2 88.9 0) (effects (font (size 1.27 1.27)) hide))
-    (property "Description" "CM4 High-Density Receptacle 1 (Power, PCIe, USB OTG, DSI/HDMI)" (at 76.2 88.9 0) (effects (font (size 1.27 1.27)) hide))
+    (property "Description" "CM5 High-Density Receptacle 1 (Power, PCIe, USB OTG, DSI/HDMI)" (at 76.2 88.9 0) (effects (font (size 1.27 1.27)) hide))
     (pin "1") ; GND
     (pin "2") ; VDD_5V
@@
     (pin "20") ; GND
   )
-  ;; J2: Hirose DF40C-100DS-0.4V (CM4 Board-to-Board Socket 2)
+  ;; J2: Hirose DF40C-100DS-0.4V (CM5 Board-to-Board Socket 2)
   (symbol (lib_id "SolarDeck_Compute:Hirose_DF40C_100DS") (at 76.2 165.1 0) (unit 1)
     (in_bom yes) (on_board yes) (dnp no)
@@
     (property "Value" "DF40C-100DS-0.4V" (at 76.2 116.84 0) (effects (font (size 1.27 1.27))))
     (property "Footprint" "Connector_Hirose:Hirose_DF40C-100DS-0.4V_2x50_P0.40mm_Vertical" (at 76.2 165.1 0) (effects (font (size 1.27 1.27)) hide))
-    (property "Description" "CM4 High-Density Receptacle 2 (GPIOs, SPI, I2C, UART, CSI Camera)" (at 76.2 165.1 0) (effects (font (size 1.27 1.27)) hide))
+    (property "Description" "CM5 High-Density Receptacle 2 (GPIOs, SPI, I2C, UART, CSI Camera)" (at 76.2 165.1 0) (effects (font (size 1.27 1.27)) hide))
     (pin "1") ; GPIO17_WAKE (from RP2350)
     (pin "2") ; GPIO16_PWRFAIL (from RP2350)
-    (pin "3") ; CM4_SPI_MOSI
-    (pin "4") ; CM4_SPI_MISO
-    (pin "5") ; CM4_SPI_SCK
-    (pin "6") ; CM4_SPI_CS
-    (pin "7") ; CM4_HRDY
-    (pin "8") ; CM4_RESET
+    (pin "3") ; CM5_SPI_MOSI
+    (pin "4") ; CM5_SPI_MISO
+    (pin "5") ; CM5_SPI_SCK
+    (pin "6") ; CM5_SPI_CS
+    (pin "7") ; CM5_HRDY
+    (pin "8") ; CM5_RESET
     (pin "9") ; UART0_TX
     (pin "10") ; UART0_RX
@@
     (pin "17") ; CAM1_D1_P
     (pin "18") ; CAM1_D1_N
-    (pin "19") ; VDD_3V3_CM4
+    (pin "19") ; VDD_3V3_CM5
     (pin "20") ; GND
   )
@@
     (pin "1") ; VDD_IO (VDD_3V3_AON)
     (pin "2") ; VDD_CORE (1.1V Internal LDO)
-    (pin "3") ; GPIO0_UART_TX (to CM4 UART0_RX)
-    (pin "4") ; GPIO1_UART_RX (to CM4 UART0_TX)
+    (pin "3") ; GPIO0_UART_TX (to CM5 UART0_RX)
+    (pin "4") ; GPIO1_UART_RX (to CM5 UART0_TX)
     (pin "5") ; GPIO2_I2C_SDA_AON
     (pin "6") ; GPIO3_I2C_SCL_AON
@@
     (pin "11") ; GPIO8_RP_HRDY (to TMUX1575 B1)
     (pin "12") ; GPIO9_RP_RESET (to TMUX1575 B1)
-    (pin "13") ; GPIO10_TMUX_SEL (0=CM4, 1=RP2350)
+    (pin "13") ; GPIO10_TMUX_SEL (0=CM5, 1=RP2350)
     (pin "14") ; GPIO11_EN_5V_SYS (Controls TPS61088)
-    (pin "15") ; GPIO12_WAKE_CM4 (<300ms S2idle wake)
-    (pin "16") ; GPIO13_PWRFAIL_CM4 (150ms flush hook)
+    (pin "15") ; GPIO12_WAKE_CM5 (<300ms S2idle wake)
+    (pin "16") ; GPIO13_PWRFAIL_CM5 (150ms flush hook)
     (pin "17") ; GPIO14_RTC_INT (1Hz DS3231 tick)
     (pin "18") ; GPIO15_CHEM_SEL (Reads SW1 strap)
@@
   (hierarchical_label "CHEM_SEL_RP" (shape input) (at 152.4 104.14 0))
   ;; Inter-Brain & Display Bus Labels
-  (hierarchical_label "CM4_SPI_MOSI" (shape output) (at 101.6 157.48 0))
-  (hierarchical_label "CM4_SPI_MISO" (shape input) (at 101.6 160.02 0))
-  (hierarchical_label "CM4_SPI_SCK" (shape output) (at 101.6 162.56 0))
-  (hierarchical_label "CM4_SPI_CS" (shape output) (at 101.6 165.1 0))
-  (hierarchical_label "CM4_HRDY" (shape input) (at 101.6 167.64 0))
-  (hierarchical_label "CM4_RESET" (shape output) (at 101.6 170.18 0))
+  (hierarchical_label "CM5_SPI_MOSI" (shape output) (at 101.6 157.48 0))
+  (hierarchical_label "CM5_SPI_MISO" (shape input) (at 101.6 160.02 0))
+  (hierarchical_label "CM5_SPI_SCK" (shape output) (at 101.6 162.56 0))
+  (hierarchical_label "CM5_SPI_CS" (shape output) (at 101.6 165.1 0))
+  (hierarchical_label "CM5_HRDY" (shape input) (at 101.6 167.64 0))
+  (hierarchical_label "CM5_RESET" (shape output) (at 101.6 170.18 0))
   (hierarchical_label "RP_SPI_MOSI" (shape output) (at 203.2 88.9 0))
   (hierarchical_label "RP_SPI_MISO" (shape input) (at 203.2 91.44 0))
@@
   (hierarchical_label "RP_HRDY" (shape input) (at 203.2 96.52 0))
   (hierarchical_label "RP_RESET" (shape output) (at 203.2 99.06 0))
-  (hierarchical_label "TMUX_SEL_CM4_NRP" (shape output) (at 203.2 104.14 0))
+  (hierarchical_label "TMUX_SEL_CM5_NRP" (shape output) (at 203.2 104.14 0))
   ;; PCIe & USB lines to I/O Sheet
   (hierarchical_label "PCIE_TX_P" (shape output) (at 101.6 78.74 0))
@@
   (hierarchical_label "PCIE_CLK_N" (shape output) (at 101.6 91.44 0))
   (hierarchical_label "PCIE_CLKREQ_L" (shape bidirectional) (at 101.6 93.98 0))
-  (hierarchical_label "CM4_USB_DP" (shape bidirectional) (at 101.6 96.52 0))
-  (hierarchical_label "CM4_USB_DM" (shape bidirectional) (at 101.6 99.06 0))
+  (hierarchical_label "CM5_USB_DP" (shape bidirectional) (at 101.6 96.52 0))
+  (hierarchical_label "CM5_USB_DM" (shape bidirectional) (at 101.6 99.06 0))
   ;; U23: BMA400 (3-Axis Accelerometer, 3.5uA pick-up wake)
   (symbol (lib_id "SolarDeck_Compute:BMA400") (at 20.0 60.0 0) (unit 1)
