File: hardware/display.kicad_sch (KiCad schematic)
At the start: 3 parts, among them U14 TMUX1575PWR, U15 SN74LVC1G08DBVR

Commit message: hardware: fix TMUX1575 fake PN (PWR->YCJR) across all artifacts; make Rule 8 scan comp values
The repo shipped TMUX1575PWR -- a part number that does not exist (TI TMUX1575
is DSBGA-YCJ only, per HARDWARE_SPEC B2/ADR-004). The fake PN was in the netlist
comp value, PCB fp_text, display sheet, BOM/CPL CSVs and both Seeed BOM exports,
while audit Rule 8 only scanned net NAMES, so the ban was silently dead code.

- parse_netlist_comps() added; Rule 8 now audits both nets and comp values
  (negative-tested: a value-embedded TMUX1575PWR is caught).
- All artifacts normalized to TMUX1575YCJR; footprint marked DSBGA-16 with dims
  TBD from TI datasheet (no fabricated package size); display sheet comment
  corrected from the banned '8-Channel' framing to 4-channel x2 devices.

Co-Authored-By: DeepSeek V4-Flash 0731 <noreply@anthropic.com>
Harness: pi (openrouter/deepseek/deepseek-v4-flash-0731, session 01a15a7c)
Parts:
- U14: value TMUX1575PWR -> TMUX1575YCJR; footprint Package_SO:TSSOP-24_4.4x7.8mm_P0.65mm -> DSBGA-16 (dims per TI datasheet; see ADR-004); symbol SolarDeck_Display:TMUX1575PWR -> SolarDeck_Display:TMUX1575YCJR
Changed lines of the file:
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@@
     (comment 2 "TMUX1575 8-Ch SPDT + IT8951 EPDC + Wacom EMR + GT911 Blanking Gate")
   )
-  ;; U14: Texas Instruments TMUX1575PWR 8-Channel SPDT High-Speed Bus Switch
-  (symbol (lib_id "SolarDeck_Display:TMUX1575PWR") (at 127.0 101.6 0) (unit 1)
+  ;; U14: Texas Instruments TMUX1575YCJR, 4-channel 2:1 SPDT display bus mux (two devices = 8 channels)
+  (symbol (lib_id "SolarDeck_Display:TMUX1575YCJR") (at 127.0 101.6 0) (unit 1)
     (in_bom yes) (on_board yes) (dnp no)
     (property "Reference" "U14" (at 127.0 58.42 0) (effects (font (size 1.27 1.27))))
-    (property "Value" "TMUX1575PWR" (at 127.0 60.96 0) (effects (font (size 1.27 1.27))))
-    (property "Footprint" "Package_SO:TSSOP-24_4.4x7.8mm_P0.65mm" (at 127.0 101.6 0) (effects (font (size 1.27 1.27)) hide))
+    (property "Value" "TMUX1575YCJR" (at 127.0 60.96 0) (effects (font (size 1.27 1.27))))
+    (property "Footprint" "DSBGA-16 (dims per TI datasheet; see ADR-004)" (at 127.0 101.6 0) (effects (font (size 1.27 1.27)) hide))
     (property "Datasheet" "https://www.ti.com/lit/ds/symlink/tmux1575.pdf" (at 127.0 101.6 0) (effects (font (size 1.27 1.27)) hide))
-    (property "Description" "8-Channel 2:1 SPDT Switch with Powered-off Protection (I_off < 10nA)" (at 127.0 101.6 0) (effects (font (size 1.27 1.27)) hide))
+    (property "Description" "4-Channel 2:1 SPDT Switch with Powered-off Protection (I_off < 10nA); two devices for 8 channels" (at 127.0 101.6 0) (effects (font (size 1.27 1.27)) hide))
     ;; Control & Power
     (pin "1") ; SEL (0 = Bank B0 CM4, 1 = Bank B1 RP2350)

Commit message: AUDIT 6 + README rewrite; standardize on CM5, Kaleido 4, SGP.22 eSIM
Class: C1 CLAIM + C4 HYGIENE (spans C2 for the overlay/identifier rename).

- docs/AUDIT_6_2026-10-21.md: repo checked against datasheets. Blockers: BQ25895
  cannot charge LiFePO4 (VREG floor 3.84 V, default 4.208 V); protector and gauge are
  Li-ion parts; CM4/CM5 have no RAM-retaining low-power state; panel/stack/cell do
  not close; schematic has no connectivity; ~half the LCSC numbers are wrong.
- README.md rewritten: intent first, pillars with real status, one status section.
- ADR-031 CM5116064 is the compute standard; ADR-032 Kaleido 4 is the only panel,
  V1 waits for release (supersedes ADR-030 two-SKU); ADR-033 soldered eSIM kept,
  must be consumer SGP.22 (ST4SIM-200M rejected).
- spec_values: panel facts, reader geometry, refresh timings, epdc_spi_mhz -> null;
  CM5 supply keys; BCM2712 (was BCM2718); BOM total re-derived as a floor.
- Gates: two dead BANNED regexes fixed (red-controlled); Phase 9 accepts any
  harness attribution and no longer claims link checking; Phases 5/10 skip null
  panel facts with an UNVERIFIED line; Phase 14 counts TBD rows; Phase 16 checks
  the CM5 commitment is stated as unpublished.
- Sweep: CM4 -> CM5 across live docs, firmware identifiers, nets, production
  guides; overlay renamed solardeck-cm5.dts and marked not yet valid (RP1 port).
- Airgap switch: ties CM5 WL_nDisable/BT_nDisable low (CM5 datasheet 2.1.1-2.1.2).

verify_all.py: 16/16 green. Still unmeasured: everything.

Co-Authored-By: Claude Opus 5.5 <noreply@anthropic.com>
Harness: claude-code (anthropic/claude-opus-5-5, session f5d955c0)
Claude-Session: https://claude.ai/code/session_01CkqVCXjctA16Vs1i2pskTP
Changed lines of the file:
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@@
     (property "Description" "4-Channel 2:1 SPDT Switch with Powered-off Protection (I_off < 10nA); two devices for 8 channels" (at 127.0 101.6 0) (effects (font (size 1.27 1.27)) hide))
     ;; Control & Power
-    (pin "1") ; SEL (0 = Bank B0 CM4, 1 = Bank B1 RP2350)
+    (pin "1") ; SEL (0 = Bank B0 CM5, 1 = Bank B1 RP2350)
     (pin "2") ; EN_L (Active LOW enable tied to GND)
     (pin "3") ; VDD (VDD_3V3_AON)
     (pin "4") ; GND
     ;; Channel 1: SPI MOSI
-    (pin "5") ; 1B0 (CM4_SPI_MOSI)
+    (pin "5") ; 1B0 (CM5_SPI_MOSI)
     (pin "6") ; 1B1 (RP_SPI_MOSI)
     (pin "7") ; 1A  (EPDC_SPI_MOSI)
     ;; Channel 2: SPI MISO
-    (pin "8") ; 2B0 (CM4_SPI_MISO)
+    (pin "8") ; 2B0 (CM5_SPI_MISO)
     (pin "9") ; 2B1 (RP_SPI_MISO)
     (pin "10") ; 2A  (EPDC_SPI_MISO)
     ;; Channel 3: SPI SCK
-    (pin "11") ; 3B0 (CM4_SPI_SCK)
+    (pin "11") ; 3B0 (CM5_SPI_SCK)
     (pin "12") ; 3B1 (RP_SPI_SCK)
     (pin "13") ; 3A  (EPDC_SPI_SCK)
     ;; Channel 4: SPI CS
-    (pin "14") ; 4B0 (CM4_SPI_CS)
+    (pin "14") ; 4B0 (CM5_SPI_CS)
     (pin "15") ; 4B1 (RP_SPI_CS)
     (pin "16") ; 4A  (EPDC_SPI_CS)
     ;; Channel 5: HRDY Status Flag
-    (pin "17") ; 5B0 (CM4_HRDY)
+    (pin "17") ; 5B0 (CM5_HRDY)
     (pin "18") ; 5B1 (RP_HRDY)
     (pin "19") ; 5A  (EPDC_HRDY)
     ;; Channel 6: RESET
-    (pin "20") ; 6B0 (CM4_RESET)
+    (pin "20") ; 6B0 (CM5_RESET)
     (pin "21") ; 6B1 (RP_RESET)
     (pin "22") ; 6A  (EPDC_RESET)
@@
     (pin "2") ; B: PEN_PROX_INT_L (Active HIGH when pen away, LOW when pen hover)
     (pin "3") ; GND
-    (pin "4") ; Y: GATED_TOUCH_INT (to CM4 GPIO)
+    (pin "4") ; Y: GATED_TOUCH_INT (to CM5 GPIO)
     (pin "5") ; VCC (VDD_3V3_AON)
   )
@@
   (hierarchical_label "VDD_3V3_AON" (shape input) (at 101.6 88.9 0))
   (hierarchical_label "VDD_5V_SYS" (shape input) (at 101.6 91.44 0))
-  (hierarchical_label "TMUX_SEL_CM4_NRP" (shape input) (at 101.6 93.98 0))
-  ;; CM4 Input Port (Bank B0)
-  (hierarchical_label "CM4_SPI_MOSI" (shape input) (at 63.5 96.52 0))
-  (hierarchical_label "CM4_SPI_MISO" (shape output) (at 63.5 99.06 0))
-  (hierarchical_label "CM4_SPI_SCK" (shape input) (at 63.5 101.6 0))
-  (hierarchical_label "CM4_SPI_CS" (shape input) (at 63.5 104.14 0))
-  (hierarchical_label "CM4_HRDY" (shape output) (at 63.5 106.68 0))
-  (hierarchical_label "CM4_RESET" (shape input) (at 63.5 109.22 0))
+  (hierarchical_label "TMUX_SEL_CM5_NRP" (shape input) (at 101.6 93.98 0))
+  ;; CM5 Input Port (Bank B0)
+  (hierarchical_label "CM5_SPI_MOSI" (shape input) (at 63.5 96.52 0))
+  (hierarchical_label "CM5_SPI_MISO" (shape output) (at 63.5 99.06 0))
+  (hierarchical_label "CM5_SPI_SCK" (shape input) (at 63.5 101.6 0))
+  (hierarchical_label "CM5_SPI_CS" (shape input) (at 63.5 104.14 0))
+  (hierarchical_label "CM5_HRDY" (shape output) (at 63.5 106.68 0))
+  (hierarchical_label "CM5_RESET" (shape input) (at 63.5 109.22 0))
   ;; RP2350 Input Port (Bank B1)
   (hierarchical_label "RP_SPI_MOSI" (shape input) (at 63.5 116.84 0))
