File: hardware/io.kicad_sch (KiCad schematic)
At the start: 5 parts, among them U16 VL805-Q6, U18 ST4SIM-200M

Commit message: schematic: capture 10 sensor/power/io BOM line items into the schematic layer (20/62 -> 30/62)
Adds U19-U28 with datasheet-anchored footprints and REAL sourced LCSC part
numbers (verified 2026-11-02): TPS22918DBVR, INA3221AIRGVR, BQ27441-G1A,
TPS2051BDBVR (power); BMA400, BMP390, TMP112AIDRLR (compute); TUSB320RWBR,
TXU0104PWR, MAX98357A (io).

Files moved in lockstep: .kicad_sch symbol blocks, netlist comps, BOM CSV rows,
CPL centroids (inside 222x160 board), kicad_pcb fp_text reference labels
(reference-grade single pads per U5/U14 convention; full pad maps and routing
remain the stated 'unrouted PCB' phase).

scripts/capture_schematic_parts.py is the generator + assert (Phase 11 contract:
netlist == BOM == CPL == 30 designators). spec_values schematic_coverage_baseline
20 -> 30; prose in README/BOM/HANDOFF normalized; STATUS.md regenerated.

Co-Authored-By: DeepSeek V4-Flash 0731 <noreply@anthropic.com>
Harness: pi (openrouter/deepseek/deepseek-v4-flash-0731, session 01a15a7c)
Parts:
- added U26: TUSB320RWBR, Package_DFN_QFN:X2QFN-12_1.6x1.6mm_P0.4mm, symbol SolarDeck_IO:TUSB320RWBR
- added U27: TXU0104PWR, Package_SO:TSSOP-14_4.4x5mm_P0.65mm, symbol SolarDeck_IO:TXU0104PWR
- added U28: MAX98357A, Package_DFN_QFN:WQFN-16-1EP_3x3mm_P0.5mm, symbol SolarDeck_IO:MAX98357A
Changed lines of the file:
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@@
   (hierarchical_label "CM4_USB_DP" (shape bidirectional) (at 50.8 114.3 0))
   (hierarchical_label "CM4_USB_DM" (shape bidirectional) (at 50.8 116.84 0))
+  ;; U26: TUSB320RWBR (USB-C Configuration Channel Dual-Role DRP Controller)
+  (symbol (lib_id "SolarDeck_IO:TUSB320RWBR") (at 140.0 60.0 0) (unit 1)
+    (in_bom yes) (on_board yes) (dnp no)
+    (property "Reference" "U26" (at 140.0 50.0 0) (effects (font (size 1.27 1.27))))
+    (property "Value" "TUSB320RWBR" (at 140.0 52.5 0) (effects (font (size 1.27 1.27))))
+    (property "Footprint" "Package_DFN_QFN:X2QFN-12_1.6x1.6mm_P0.4mm" (at 140.0 60.0 0) (effects (font (size 1.27 1.27)) hide))
+    (property "Datasheet" "https://www.ti.com/lit/ds/symlink/tusb320.pdf" (at 140.0 60.0 0) (effects (font (size 1.27 1.27)) hide))
+    (property "Description" "USB-C Configuration Channel Dual-Role DRP Controller" (at 140.0 60.0 0) (effects (font (size 1.27 1.27)) hide))
+  )
+  ;; U27: TXU0104PWR (Fail-Safe Cross-Domain Buffer with I_off Partial-Power-Down)
+  (symbol (lib_id "SolarDeck_IO:TXU0104PWR") (at 155.0 60.0 0) (unit 1)
+    (in_bom yes) (on_board yes) (dnp no)
+    (property "Reference" "U27" (at 155.0 50.0 0) (effects (font (size 1.27 1.27))))
+    (property "Value" "TXU0104PWR" (at 155.0 52.5 0) (effects (font (size 1.27 1.27))))
+    (property "Footprint" "Package_SO:TSSOP-14_4.4x5mm_P0.65mm" (at 155.0 60.0 0) (effects (font (size 1.27 1.27)) hide))
+    (property "Datasheet" "https://www.ti.com/lit/ds/symlink/txu0104.pdf" (at 155.0 60.0 0) (effects (font (size 1.27 1.27)) hide))
+    (property "Description" "Fail-Safe Cross-Domain Buffer with I_off Partial-Power-Down" (at 155.0 60.0 0) (effects (font (size 1.27 1.27)) hide))
+  )
+  ;; U28: MAX98357A (I2S Class-D Speaker Amplifier, 1W)
+  (symbol (lib_id "SolarDeck_IO:MAX98357A") (at 170.0 60.0 0) (unit 1)
+    (in_bom yes) (on_board yes) (dnp no)
+    (property "Reference" "U28" (at 170.0 50.0 0) (effects (font (size 1.27 1.27))))
+    (property "Value" "MAX98357A" (at 170.0 52.5 0) (effects (font (size 1.27 1.27))))
+    (property "Footprint" "Package_DFN_QFN:WQFN-16-1EP_3x3mm_P0.5mm" (at 170.0 60.0 0) (effects (font (size 1.27 1.27)) hide))
+    (property "Datasheet" "https://www.analog.com/media/en/technical-datasheets/max98357a.pdf" (at 170.0 60.0 0) (effects (font (size 1.27 1.27)) hide))
+    (property "Description" "I2S Class-D Speaker Amplifier, 1W (MAX98357A)" (at 170.0 60.0 0) (effects (font (size 1.27 1.27)) hide))
+  )
 )

Commit message: schematic: capture 10 more BOM line items (30/62 -> 40/62) with real LCSC numbers
Batch 2: STUSB4500QTR (PD sink), BQ29700DSET (battery PCM), LM66100DCKR (VBUS
OR-ing), PN5321A3HN (NFC + crypto signer), TPD4E05U06 (ESD TVS), dual
SPH0645LM4H-B (MEMS beamforming pair at 65mm), E22-900M22S (LoRa), PCM5102APWR
(headphone DAC), DRV2605LDGST (haptic).

Footprints datasheet-anchored, incl. corrections the searches caught (TPD4E05
is USON-10 not SOT-23-6, LM66100 is SC-70-6, PCM5102A is TSSOP-20, DRV2605L is
VSSOP-10). capture_schematic_parts.py now also emits kicad_pcb footprint blocks
(reference-grade single pad per U5/U14 convention) and is fully idempotent.
Phase 11 guard extended: live prose restatements must match the netlist.

spec_values baseline 30 -> 40; README/HANDOFF prose normalized; STATUS regenerated.

Co-Authored-By: DeepSeek V4-Flash 0731 <noreply@anthropic.com>
Harness: pi (openrouter/deepseek/deepseek-v4-flash-0731, session 01a15a7c)
Parts:
- added U30: PN5321A3HN, Package_DFN_QFN:HVQFN-40_6x6mm_P0.5mm, symbol SolarDeck_IO:PN5321A3HN
- added U33: TPD4E05U06, Package_DFN_QFN:USON-10_2.5x1mm_P0.5mm, symbol SolarDeck_IO:TPD4E05U06
- added U34, U35: SPH0645LM4H-B, Package_LGA:MIC-SMD-6P_3.5x2.65mm_P0.9mm, symbol SolarDeck_IO:SPH0645LM4H-B
- added U36: E22-900M22S, Module_EByte:E22-900M22S_20x14mm, symbol SolarDeck_IO:E22-900M22S
- added U37: PCM5102APWR, Package_SO:TSSOP-20_6.5x4.4mm_P0.65mm, symbol SolarDeck_IO:PCM5102APWR
- added U38: DRV2605LDGST, Package_TO_SOT_SMD:VSSOP-10_3x4.9mm_P0.5mm, symbol SolarDeck_IO:DRV2605LDGST
Changed lines of the file:
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@@
     (property "Description" "I2S Class-D Speaker Amplifier, 1W (MAX98357A)" (at 170.0 60.0 0) (effects (font (size 1.27 1.27)) hide))
   )
+  ;; U30: PN5321A3HN (13.56MHz NFC/Smartcard Controller + Crypto Signer)
+  (symbol (lib_id "SolarDeck_IO:PN5321A3HN") (at 20.0 80.0 0) (unit 1)
+    (in_bom yes) (on_board yes) (dnp no)
+    (property "Reference" "U30" (at 20.0 70.0 0) (effects (font (size 1.27 1.27))))
+    (property "Value" "PN5321A3HN" (at 20.0 72.5 0) (effects (font (size 1.27 1.27))))
+    (property "Footprint" "Package_DFN_QFN:HVQFN-40_6x6mm_P0.5mm" (at 20.0 80.0 0) (effects (font (size 1.27 1.27)) hide))
+    (property "Datasheet" "https://www.nxp.com/docs/en/data-sheet/PN5321A3-C10655.pdf" (at 20.0 80.0 0) (effects (font (size 1.27 1.27)) hide))
+    (property "Description" "13.56MHz NFC/Smartcard Controller + Crypto Signer (FeliCa/ISO14443)" (at 20.0 80.0 0) (effects (font (size 1.27 1.27)) hide))
+  )
+  ;; U33: TPD4E05U06 (Low-Capacitance ESD/TVS Diode Array)
+  (symbol (lib_id "SolarDeck_IO:TPD4E05U06") (at 50.0 80.0 0) (unit 1)
+    (in_bom yes) (on_board yes) (dnp no)
+    (property "Reference" "U33" (at 50.0 70.0 0) (effects (font (size 1.27 1.27))))
+    (property "Value" "TPD4E05U06" (at 50.0 72.5 0) (effects (font (size 1.27 1.27))))
+    (property "Footprint" "Package_DFN_QFN:USON-10_2.5x1mm_P0.5mm" (at 50.0 80.0 0) (effects (font (size 1.27 1.27)) hide))
+    (property "Datasheet" "https://www.ti.com/lit/ds/symlink/tpd4e05u06.pdf" (at 50.0 80.0 0) (effects (font (size 1.27 1.27)) hide))
+    (property "Description" "Low-Capacitance ESD/TVS Diode Array (USB-C pin protection)" (at 50.0 80.0 0) (effects (font (size 1.27 1.27)) hide))
+  )
+  ;; U34: SPH0645LM4H-B (I2S Digital MEMS Microphone)
+  (symbol (lib_id "SolarDeck_IO:SPH0645LM4H-B") (at 110.0 80.0 0) (unit 1)
+    (in_bom yes) (on_board yes) (dnp no)
+    (property "Reference" "U34" (at 110.0 70.0 0) (effects (font (size 1.27 1.27))))
+    (property "Value" "SPH0645LM4H-B" (at 110.0 72.5 0) (effects (font (size 1.27 1.27))))
+    (property "Footprint" "Package_LGA:MIC-SMD-6P_3.5x2.65mm_P0.9mm" (at 110.0 80.0 0) (effects (font (size 1.27 1.27)) hide))
+    (property "Datasheet" "https://www.knowles.com/docs/default-source/knowles-datasheets/SPH0645LM4H-B_datasheet.pdf" (at 110.0 80.0 0) (effects (font (size 1.27 1.27)) hide))
+    (property "Description" "I2S Digital MEMS Microphone (left, 65mm from U35)" (at 110.0 80.0 0) (effects (font (size 1.27 1.27)) hide))
+  )
+  ;; U35: SPH0645LM4H-B (I2S Digital MEMS Microphone)
+  (symbol (lib_id "SolarDeck_IO:SPH0645LM4H-B") (at 175.0 80.0 0) (unit 1)
+    (in_bom yes) (on_board yes) (dnp no)
+    (property "Reference" "U35" (at 175.0 70.0 0) (effects (font (size 1.27 1.27))))
+    (property "Value" "SPH0645LM4H-B" (at 175.0 72.5 0) (effects (font (size 1.27 1.27))))
+    (property "Footprint" "Package_LGA:MIC-SMD-6P_3.5x2.65mm_P0.9mm" (at 175.0 80.0 0) (effects (font (size 1.27 1.27)) hide))
+    (property "Datasheet" "https://www.knowles.com/docs/default-source/knowles-datasheets/SPH0645LM4H-B_datasheet.pdf" (at 175.0 80.0 0) (effects (font (size 1.27 1.27)) hide))
+    (property "Description" "I2S Digital MEMS Microphone (right, 65mm from U34)" (at 175.0 80.0 0) (effects (font (size 1.27 1.27)) hide))
+  )
+  ;; U36: E22-900M22S (915/868MHz LoRa Transceiver Module)
+  (symbol (lib_id "SolarDeck_IO:E22-900M22S") (at 20.0 110.0 0) (unit 1)
+    (in_bom yes) (on_board yes) (dnp no)
+    (property "Reference" "U36" (at 20.0 100.0 0) (effects (font (size 1.27 1.27))))
+    (property "Value" "E22-900M22S" (at 20.0 102.5 0) (effects (font (size 1.27 1.27))))
+    (property "Footprint" "Module_EByte:E22-900M22S_20x14mm" (at 20.0 110.0 0) (effects (font (size 1.27 1.27)) hide))
+    (property "Datasheet" "https://www.ebyte.com/en/product-view-news.html?id=1569" (at 20.0 110.0 0) (effects (font (size 1.27 1.27)) hide))
+    (property "Description" "915/868MHz LoRa Transceiver Module (Semtech SX1262, +22dBm)" (at 20.0 110.0 0) (effects (font (size 1.27 1.27)) hide))
+  )
+  ;; U37: PCM5102APWR (32-bit Stereo I2S Headphone DAC)
+  (symbol (lib_id "SolarDeck_IO:PCM5102APWR") (at 155.0 110.0 0) (unit 1)
+    (in_bom yes) (on_board yes) (dnp no)
+    (property "Reference" "U37" (at 155.0 100.0 0) (effects (font (size 1.27 1.27))))
+    (property "Value" "PCM5102APWR" (at 155.0 102.5 0) (effects (font (size 1.27 1.27))))
+    (property "Footprint" "Package_SO:TSSOP-20_6.5x4.4mm_P0.65mm" (at 155.0 110.0 0) (effects (font (size 1.27 1.27)) hide))
+    (property "Datasheet" "https://www.ti.com/lit/ds/symlink/pcm5102a.pdf" (at 155.0 110.0 0) (effects (font (size 1.27 1.27)) hide))
+    (property "Description" "32-bit Stereo I2S Headphone DAC (384kHz)" (at 155.0 110.0 0) (effects (font (size 1.27 1.27)) hide))
+  )
+  ;; U38: DRV2605LDGST (Wideband Haptic Driver)
+  (symbol (lib_id "SolarDeck_IO:DRV2605LDGST") (at 170.0 110.0 0) (unit 1)
+    (in_bom yes) (on_board yes) (dnp no)
+    (property "Reference" "U38" (at 170.0 100.0 0) (effects (font (size 1.27 1.27))))
+    (property "Value" "DRV2605LDGST" (at 170.0 102.5 0) (effects (font (size 1.27 1.27))))
+    (property "Footprint" "Package_TO_SOT_SMD:VSSOP-10_3x4.9mm_P0.5mm" (at 170.0 110.0 0) (effects (font (size 1.27 1.27)) hide))
+    (property "Datasheet" "https://www.ti.com/lit/ds/symlink/drv2605l.pdf" (at 170.0 110.0 0) (effects (font (size 1.27 1.27)) hide))
+    (property "Description" "Wideband Haptic Driver (LRA actuator controller)" (at 170.0 110.0 0) (effects (font (size 1.27 1.27)) hide))
+  )
 )

Commit message: AUDIT 6 + README rewrite; standardize on CM5, Kaleido 4, SGP.22 eSIM
Class: C1 CLAIM + C4 HYGIENE (spans C2 for the overlay/identifier rename).

- docs/AUDIT_6_2026-10-21.md: repo checked against datasheets. Blockers: BQ25895
  cannot charge LiFePO4 (VREG floor 3.84 V, default 4.208 V); protector and gauge are
  Li-ion parts; CM4/CM5 have no RAM-retaining low-power state; panel/stack/cell do
  not close; schematic has no connectivity; ~half the LCSC numbers are wrong.
- README.md rewritten: intent first, pillars with real status, one status section.
- ADR-031 CM5116064 is the compute standard; ADR-032 Kaleido 4 is the only panel,
  V1 waits for release (supersedes ADR-030 two-SKU); ADR-033 soldered eSIM kept,
  must be consumer SGP.22 (ST4SIM-200M rejected).
- spec_values: panel facts, reader geometry, refresh timings, epdc_spi_mhz -> null;
  CM5 supply keys; BCM2712 (was BCM2718); BOM total re-derived as a floor.
- Gates: two dead BANNED regexes fixed (red-controlled); Phase 9 accepts any
  harness attribution and no longer claims link checking; Phases 5/10 skip null
  panel facts with an UNVERIFIED line; Phase 14 counts TBD rows; Phase 16 checks
  the CM5 commitment is stated as unpublished.
- Sweep: CM4 -> CM5 across live docs, firmware identifiers, nets, production
  guides; overlay renamed solardeck-cm5.dts and marked not yet valid (RP1 port).
- Airgap switch: ties CM5 WL_nDisable/BT_nDisable low (CM5 datasheet 2.1.1-2.1.2).

verify_all.py: 16/16 green. Still unmeasured: everything.

Co-Authored-By: Claude Opus 5.5 <noreply@anthropic.com>
Harness: claude-code (anthropic/claude-opus-5-5, session f5d955c0)
Claude-Session: https://claude.ai/code/session_01CkqVCXjctA16Vs1i2pskTP
Changed lines of the file:
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@@
   (hierarchical_label "VDD_5V_SYS" (shape input) (at 50.8 78.74 0))
   (hierarchical_label "VDD_3V8_MODEM" (shape input) (at 152.4 76.2 0))
-  ;; PCIe Upstream from CM4
+  ;; PCIe Upstream from CM5
   (hierarchical_label "PCIE_TX_P" (shape input) (at 50.8 88.9 0))
   (hierarchical_label "PCIE_TX_N" (shape input) (at 50.8 91.44 0))
@@
   (hierarchical_label "PCIE_CLKREQ_L" (shape bidirectional) (at 50.8 104.14 0))
   ;; USB-C Native Port 1
-  (hierarchical_label "CM4_USB_DP" (shape bidirectional) (at 50.8 114.3 0))
-  (hierarchical_label "CM4_USB_DM" (shape bidirectional) (at 50.8 116.84 0))
+  (hierarchical_label "CM5_USB_DP" (shape bidirectional) (at 50.8 114.3 0))
+  (hierarchical_label "CM5_USB_DM" (shape bidirectional) (at 50.8 116.84 0))
   ;; U26: TUSB320RWBR (USB-C Configuration Channel Dual-Role DRP Controller)
   (symbol (lib_id "SolarDeck_IO:TUSB320RWBR") (at 140.0 60.0 0) (unit 1)
